Commit message: updated yaml

File: nuturtle_description/urdf/turtlebot3_burger.urdf.xacro (robot description, xacro)
@@ -2,4 +2,12 @@
 <robot name="turtlebot3_burger"
   xmlns:xacro="http://ros.org/wiki/xacro">
+<xacro:property name="prop" value="${xacro.load_yaml('$(find nuturtle_description)/diff_params.yaml')['/**']
+['ros__parameters']}"/>
+<xacro:property name="wheel_radius" value="${prop['wheel_radius']}"/>
+<xacro:property name="track_width" value="${prop['track_width']}"/>
+<xacro:property name="motor_cmd_max" value="${prop['motor_cmd_max']}"/>
+<xacro:property name="motor_cmd_per_rad_sec" value="${prop['motor_cmd_per_rad_sec']}"/>
+<xacro:property name="encoder_ticks_per_rad" value="${prop['encoder_ticks_per_rad']}"/>
+<xacro:property name="collision_radius" value="${prop['collision_radius']}"/>
   <!-- <xacro:include filename="$(find turtlebot3_description)/urdf/common_properties.urdf"/> -->
   <!-- Init colour -->

Commit message: added A.4 features

File: nuturtle_description/urdf/turtlebot3_burger.urdf.xacro (robot description, xacro)
@@ -2,4 +2,5 @@
 <robot name="turtlebot3_burger"
   xmlns:xacro="http://ros.org/wiki/xacro">
+<xacro:arg name="color" default="purple"/>
 <xacro:property name="prop" value="${xacro.load_yaml('$(find nuturtle_description)/diff_params.yaml')['/**']
 ['ros__parameters']}"/>
@@ -36,4 +37,7 @@
     <color rgba="1.0 1.0 1.0 1.0"/>
   </material>
+  <material name="purple">
+    <color rgba="0.3 0.16 0.52 1.0"/>
+  </material>
   <link name="base_footprint"/>
   <joint name="base_joint" type="fixed">
@@ -46,17 +50,17 @@
       <origin xyz="-0.032 0 0.0" rpy="0 0 0"/>
       <geometry>
+          <mesh filename="file://$(find nuturtle_description)/burger_base.stl" scale="0.001 0.001 0.001"/>
+      </geometry>
+      <material name="$(arg color)"/>
+    </visual>
+    <collision>
+      <origin xyz="-0.032 0 0.070" rpy="0 0 0"/>
+      <geometry>
         <xacro:if value="${collision_radius&gt;0}">
           <cylinder radius="${collision_radius}" length="0.081"/>
         </xacro:if>
         <xacro:if value="${collision_radius&lt;0}">
-          <mesh filename="file://$(find nuturtle_description)/burger_base.stl" scale="0.001 0.001 0.001"/>
+          <box size="0.140 0.140 0.143"/>
         </xacro:if>
-      </geometry>
-      <material name="light_black"/>
-    </visual>
-    <collision>
-      <origin xyz="-0.032 0 0.070" rpy="0 0 0"/>
-      <geometry>
-        <box size="0.140 0.140 0.143"/>
       </geometry>
     </collision>

Commit message: launch file doesnt work

File: nuturtle_description/urdf/turtlebot3_burger.urdf.xacro (robot description, xacro)
@@ -81,5 +81,5 @@
       <origin xyz="0 0 0" rpy="1.57 0 0"/>
       <geometry>
-        <mesh filename="file://$(find nuturtle_description)/left_tire.stl" scale="${wheel_radius} 0.001 ${wheel_radius}"/>
+        <mesh filename="file://$(find nuturtle_description)/left_tire.stl" scale="0.001 0.001 0.001"/>
       </geometry>
       <material name="dark"/>
@@ -88,5 +88,5 @@
       <origin xyz="0 0 0" rpy="0 0 0"/>
       <geometry>
-        <cylinder length="0.018" radius="0.033"/>
+        <cylinder length="0.018" radius="${wheel_radius}"/>
       </geometry>
     </collision>
@@ -107,5 +107,5 @@
       <origin xyz="0 0 0" rpy="1.57 0 0"/>
       <geometry>
-        <mesh filename="file://$(find nuturtle_description)/right_tire.stl" scale="${wheel_radius} 0.001 ${wheel_radius}"/>
+        <mesh filename="file://$(find nuturtle_description)/right_tire.stl" scale="0.001 0.001 0.001"/>
       </geometry>
       <material name="dark"/>
@@ -114,5 +114,5 @@
       <origin xyz="0 0 0" rpy="0 0 0"/>
       <geometry>
-        <cylinder length="0.018" radius="0.033"/>
+        <cylinder length="0.018" radius="${wheel_radius}"/>
       </geometry>
     </collision>
